File: hardware/STM32F042F6P6-tryout.sch (KiCad schematic (older format))
At the start: 26 parts

Commit message: update,
Parts:
- removed FB?: UPZ1608E221-2R2TF, symbol taobao-bead:Ferrite_Bead_Small
- added FB1: UPZ1608E221-2R2TF, Inductor_SMD:L_0603_1608Metric_Pad1.05x0.95mm_HandSolder, symbol taobao-components:UPZ1608E221-2R2TF
- J1: renamed from J?; footprint (none) -> Connector_USB:USB_Micro-B_Molex_47346-0001
- J2: renamed from J?; footprint (none) -> Connector_PinHeader_2.54mm:PinHeader_2x02_P2.54mm_Vertical
- U4: renamed from U?; footprint (none) -> Connector_PinHeader_2.54mm:PinHeader_1x03_P2.54mm_Vertical
- gave numbers to parts that had none: 22
Connections:
- net +5V: now also FB1.1
- net at C3.1, J1.1 (VBUS), U2.5 (VBUS): now also FB1.2
Other:
- note added: "? internal pull up \nresistor from stm32 ?"
